File: v0_miniAB_pancake_board.kicad_sch (KiCad schematic)
At the start: 11 parts, among them J1 Conn_01x04_Female, J2 Conn_01x02_Female, J3 Conn_01x02_Female, J4 Conn_01x02_Female, J5 Conn_01x02_Female, J6 Conn_01x02_Female, J7 Conn_01x03_Female, J8 Conn_01x03_Female, J9 Conn_02x07_Counter_Clockwise

Commit message: First steps of the batboard conversion
Parts:
- J9: footprint Connector_Molex:Molex_Micro-Fit_3.0_43045-1400_2x07_P3.00mm_Horizontal -> Connector_Molex:Molex_Micro-Fit_3.0_43045-1800_2x09_P3.00mm_Horizontal; symbol Connector_Generic:Conn_02x07_Top_Bottom -> Connector_Generic:Conn_02x09_Top_Bottom
- J?: renamed from J3; value Conn_01x02_Female -> Conn_01x04_Female; symbol Connector:Conn_01x02_Female -> Connector:Conn_01x04_Female
- gave numbers to parts that had none: 2
Connections:
- net +24V: now also J9.11 (Pin_11); no longer J9.8 (Pin_8)
- net +5V: now also J9.17 (Pin_17); no longer J9.14 (Pin_14)
- net A+: now also J9.2 (Pin_2); no longer J9.1 (Pin_1)
- net A-: now also J9.3 (Pin_3); no longer J9.2 (Pin_2)
- net B+: now also J9.4 (Pin_4); no longer J9.3 (Pin_3)
- net B-: now also J9.5 (Pin_5); no longer J9.4 (Pin_4)
- net GND: now also J9.8 (Pin_8); no longer J9.7 (Pin_7)
- net fan0: now also J9.7 (Pin_7); no longer J9.6 (Pin_6)
- net fan1: now also J9.16 (Pin_16); no longer J9.13 (Pin_13)
- net heat_gnd: now also J9.12 (Pin_12); no longer J9.9 (Pin_9)
- net sw0: now also J9.15 (Pin_15); no longer J9.12 (Pin_12)
- net sw1: now also J9.6 (Pin_6); no longer J9.5 (Pin_5)
- net therm0: now also J9.13 (Pin_13); no longer J9.10 (Pin_10)
- net therm1: now also J9.14 (Pin_14); no longer J9.11 (Pin_11)
Changed lines of the file:
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@@
     (stroke (width 0) (type default) (color 0 0 0 0))
   )
-  (wire (pts (xy 45.72 34.29) (xy 57.15 34.29))
+  (wire (pts (xy 44.45 34.29) (xy 57.15 34.29))
     (stroke (width 0) (type default) (color 0 0 0 0))
   )
@@
     (stroke (width 0) (type default) (color 0 0 0 0))
   )
-  (wire (pts (xy 45.72 36.83) (xy 57.15 36.83))
+  (wire (pts (xy 44.45 36.83) (xy 57.15 36.83))
     (stroke (width 0) (type default) (color 0 0 0 0))
   )
@@
     (pin "2")
   )
-  (symbol (lib_id "Connector:Conn_01x02_Female") (at 40.64 34.29 0) (mirror y) (unit 1)
-    (in_bom yes) (on_board yes)
-    (property "Reference" "J3" (id 0) (at 39.9288 34.8996 0)
-      (effects (font (size 1.27 1.27)) (justify left))
-    )
-    (property "Value" "Conn_01x02_Female" (id 1) (at 39.9288 37.211 0)
-      (effects (font (size 1.27 1.27)) (justify left))
-    )
-    (property "Footprint" "Connector_JST:JST_PH_B2B-PH-K_1x02_P2.00mm_Vertical" (id 2) (at 40.64 34.29 0)
-      (effects (font (size 1.27 1.27)) hide)
-    )
-    (property "Datasheet" "~" (id 3) (at 40.64 34.29 0)
-      (effects (font (size 1.27 1.27)) hide)
-    )
-    (pin "1")
-    (pin "2")
+  (symbol (lib_id "Connector:Conn_01x04_Female") (at 39.37 36.83 0) (mirror y) (unit 1)
+    (in_bom yes) (on_board yes)
+    (property "Reference" "J?" (id 0) (at 39.37 31.75 0))
+    (property "Value" "Conn_01x04_Female" (id 1) (at 39.37 44.45 0))
+    (property "Footprint" "Connector_JST:JST_PH_B2B-PH-K_1x02_P2.00mm_Vertical" (id 2) (at 39.37 36.83 0)
+      (effects (font (size 1.27 1.27)) hide)
+    )
+    (property "Datasheet" "~" (id 3) (at 39.37 36.83 0)
+      (effects (font (size 1.27 1.27)) hide)
+    )
+    (pin "1")
+    (pin "2")
+    (pin "3")
+    (pin "4")
   )
   (symbol (lib_id "Connector:Conn_01x03_Female") (at 71.12 33.02 0) (mirror y) (unit 1)
@@
     (pin "1")
   )
-  (symbol (lib_id "Connector_Generic:Conn_02x07_Top_Bottom") (at 133.35 31.75 0) (unit 1)
+  (symbol (lib_id "Connector_Generic:Conn_02x09_Top_Bottom") (at 133.35 31.75 0) (unit 1)
     (in_bom yes) (on_board yes)
     (property "Reference" "J9" (id 0) (at 134.62 18.6182 0))
-    (property "Value" "Conn_02x07_Counter_Clockwise" (id 1) (at 134.62 20.9296 0))
-    (property "Footprint" "Connector_Molex:Molex_Micro-Fit_3.0_43045-1400_2x07_P3.00mm_Horizontal" (id 2) (at 133.35 31.75 0)
+    (property "Value" "Conn_02x07_Counter_Clockwise" (id 1) (at 134.62 16.51 0))
+    (property "Footprint" "Connector_Molex:Molex_Micro-Fit_3.0_43045-1800_2x09_P3.00mm_Horizontal" (id 2) (at 133.35 31.75 0)
       (effects (font (size 1.27 1.27)) hide)
     )
@@
     (pin "13")
     (pin "14")
+    (pin "15")
+    (pin "16")
+    (pin "17")
+    (pin "18")
     (pin "2")
     (pin "3")
@@
   (symbol (lib_id "power:+24V") (at 152.4 24.13 0) (unit 1)
     (in_bom yes) (on_board yes)
-    (property "Reference" "#PWR?" (id 0) (at 152.4 27.94 0)
+    (property "Reference" "#PWR0105" (id 0) (at 152.4 27.94 0)
       (effects (font (size 1.27 1.27)) hide)
     )
@@
   (symbol (lib_id "power:+24V") (at 57.15 26.67 0) (unit 1)
     (in_bom yes) (on_board yes)
-    (property "Reference" "#PWR?" (id 0) (at 57.15 30.48 0)
+    (property "Reference" "#PWR0106" (id 0) (at 57.15 30.48 0)
       (effects (font (size 1.27 1.27)) hide)
     )
@@
   (symbol (lib_id "Connector:Conn_01x03_Female") (at 81.28 81.28 0) (mirror y) (unit 1)
     (in_bom yes) (on_board yes)
-    (property "Reference" "J?" (id 0) (at 84.0232 74.041 0))
+    (property "Reference" "J10" (id 0) (at 84.0232 74.041 0))
     (property "Value" "Conn_01x03_Female" (id 1) (at 84.0232 76.3524 0))
     (property "Footprint" "Jumper:SolderJumper-3_P1.3mm_Bridged12_RoundedPad1.0x1.5mm_NumberLabels" (id 2) (at 81.28 81.28 0)
@@
   (symbol (lib_id "power:+5V") (at 97.79 77.47 0) (unit 1)
     (in_bom yes) (on_board yes)
-    (property "Reference" "#PWR?" (id 0) (at 97.79 81.28 0)
+    (property "Reference" "#PWR0103" (id 0) (at 97.79 81.28 0)
       (effects (font (size 1.27 1.27)) hide)
     )
@@
   (symbol (lib_id "power:+24V") (at 102.87 77.47 0) (unit 1)
     (in_bom yes) (on_board yes)
-    (property "Reference" "#PWR?" (id 0) (at 102.87 81.28 0)
+    (property "Reference" "#PWR0104" (id 0) (at 102.87 81.28 0)
       (effects (font (size 1.27 1.27)) hide)
     )
@@
   (symbol (lib_id "Connector:Conn_01x03_Female") (at 81.28 96.52 0) (mirror y) (unit 1)
     (in_bom yes) (on_board yes)
-    (property "Reference" "J?" (id 0) (at 84.0232 89.281 0))
+    (property "Reference" "J11" (id 0) (at 84.0232 89.281 0))
     (property "Value" "Conn_01x03_Female" (id 1) (at 84.0232 91.5924 0))
     (property "Footprint" "Jumper:SolderJumper-3_P1.3mm_Bridged12_RoundedPad1.0x1.5mm_NumberLabels" (id 2) (at 81.28 96.52 0)
@@
   (symbol (lib_id "power:+5V") (at 97.79 92.71 0) (unit 1)
     (in_bom yes) (on_board yes)
-    (property "Reference" "#PWR?" (id 0) (at 97.79 96.52 0)
+    (property "Reference" "#PWR0101" (id 0) (at 97.79 96.52 0)
       (effects (font (size 1.27 1.27)) hide)
     )
@@
   (symbol (lib_id "power:+24V") (at 102.87 92.71 0) (unit 1)
     (in_bom yes) (on_board yes)
-    (property "Reference" "#PWR?" (id 0) (at 102.87 96.52 0)
+    (property "Reference" "#PWR0102" (id 0) (at 102.87 96.52 0)
       (effects (font (size 1.27 1.27)) hide)
     )
@@
       (reference "#PWR09") (unit 1) (value "+5V") (footprint "")
     )
+    (path "/00000000-0000-0000-0000-0000612c7acb"
+      (reference "#PWR0101") (unit 1) (value "+5V") (footprint "")
+    )
+    (path "/00000000-0000-0000-0000-0000612c7ad7"
+      (reference "#PWR0102") (unit 1) (value "+24V") (footprint "")
+    )
+    (path "/00000000-0000-0000-0000-0000612c2dd0"
+      (reference "#PWR0103") (unit 1) (value "+5V") (footprint "")
+    )
+    (path "/00000000-0000-0000-0000-0000612c4406"
+      (reference "#PWR0104") (unit 1) (value "+24V") (footprint "")
+    )
     (path "/00000000-0000-0000-0000-0000612b9e54"
-      (reference "#PWR?") (unit 1) (value "+24V") (footprint "")
+      (reference "#PWR0105") (unit 1) (value "+24V") (footprint "")
     )
     (path "/00000000-0000-0000-0000-0000612bf736"
-      (reference "#PWR?") (unit 1) (value "+24V") (footprint "")
-    )
-    (path "/00000000-0000-0000-0000-0000612c2dd0"
-      (reference "#PWR?") (unit 1) (value "+5V") (footprint "")
-    )
-    (path "/00000000-0000-0000-0000-0000612c4406"
-      (reference "#PWR?") (unit 1) (value "+24V") (footprint "")
-    )
-    (path "/00000000-0000-0000-0000-0000612c7acb"
-      (reference "#PWR?") (unit 1) (value "+5V") (footprint "")
-    )
-    (path "/00000000-0000-0000-0000-0000612c7ad7"
-      (reference "#PWR?") (unit 1) (value "+24V") (footprint "")
+      (reference "#PWR0106") (unit 1) (value "+24V") (footprint "")
     )
     (path "/00000000-0000-0000-0000-000060d55abc"
@@
       (reference "J2") (unit 1) (value "Conn_01x02_Female") (footprint "Connector_Molex:Molex_Micro-Fit_3.0_43045-0200_2x01_P3.00mm_Horizontal")
     )
-    (path "/00000000-0000-0000-0000-000060d4eb4a"
-      (reference "J3") (unit 1) (value "Conn_01x02_Female") (footprint "Connector_JST:JST_PH_B2B-PH-K_1x02_P2.00mm_Vertical")
-    )
     (path "/00000000-0000-0000-0000-000060d4bb3b"
       (reference "J4") (unit 1) (value "Conn_01x02_Female") (footprint "Connector_JST:JST_PH_B2B-PH-K_1x02_P2.00mm_Vertical")
@@
     )
     (path "/00000000-0000-0000-0000-000060d59db3"
-      (reference "J9") (unit 1) (value "Conn_02x07_Counter_Clockwise") (footprint "Connector_Molex:Molex_Micro-Fit_3.0_43045-1400_2x07_P3.00mm_Horizontal")
+      (reference "J9") (unit 1) (value "Conn_02x07_Counter_Clockwise") (footprint "Connector_Molex:Molex_Micro-Fit_3.0_43045-1800_2x09_P3.00mm_Horizontal")
     )
     (path "/00000000-0000-0000-0000-0000612c0080"
-      (reference "J?") (unit 1) (value "Conn_01x03_Female") (footprint "Jumper:SolderJumper-3_P1.3mm_Bridged12_RoundedPad1.0x1.5mm_NumberLabels")
+      (reference "J10") (unit 1) (value "Conn_01x03_Female") (footprint "Jumper:SolderJumper-3_P1.3mm_Bridged12_RoundedPad1.0x1.5mm_NumberLabels")
     )
     (path "/00000000-0000-0000-0000-0000612c7ac0"
-      (reference "J?") (unit 1) (value "Conn_01x03_Female") (footprint "Jumper:SolderJumper-3_P1.3mm_Bridged12_RoundedPad1.0x1.5mm_NumberLabels")
-    )
-  )
+      (reference "J11") (unit 1) (value "Conn_01x03_Female") (footprint "Jumper:SolderJumper-3_P1.3mm_Bridged12_RoundedPad1.0x1.5mm_NumberLabels")
+    )
+    (path "/00000000-0000-0000-0000-000060d4eb4a"
+      (reference "J?") (unit 1) (value "Conn_01x04_Female") (footprint "Connector_JST:JST_PH_B2B-PH-K_1x02_P2.00mm_Vertical")
+    )
+  )

Commit message: Further connections made
Parts:
- J3: renamed from J?; footprint Connector_JST:JST_PH_B2B-PH-K_1x02_P2.00mm_Vertical -> Connector_JST:JST_PH_B4B-PH-K_1x04_P2.00mm_Vertical
Connections:
- net fan1: now also J9.18 (Pin_18); no longer J9.16 (Pin_16)
- net sw0: now also J9.9 (Pin_9); no longer J9.15 (Pin_15)
- net therm2: now reaches J3.3 (Pin_3)
- net therm2: now also J9.16 (Pin_16)
- net therm3: now reaches J3.4 (Pin_4)
- net therm3: now also J9.15 (Pin_15)
Changed lines of the file:
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@@
+    (stroke (width 0) (type default) (color 0 0 0 0))
+  )
+  (wire (pts (xy 140.97 41.91) (xy 152.4 41.91))
     (stroke (width 0) (type default) (color 0 0 0 0))
   )
@@
     (stroke (width 0) (type default) (color 0 0 0 0))
   )
+  (wire (pts (xy 116.84 41.91) (xy 128.27 41.91))
+    (stroke (width 0) (type default) (color 0 0 0 0))
+  )
   (wire (pts (xy 128.27 39.37) (xy 118.11 39.37))
     (stroke (width 0) (type default) (color 0 0 0 0))
   )
+  (wire (pts (xy 76.2 35.56) (xy 87.63 35.56))
+    (stroke (width 0) (type default) (color 0 0 0 0))
+  )
+  (wire (pts (xy 49.53 55.88) (xy 57.15 55.88))
+    (stroke (width 0) (type default) (color 0 0 0 0))
+  )
+  (wire (pts (xy 45.72 78.74) (xy 57.15 78.74))
+    (stroke (width 0) (type default) (color 0 0 0 0))
+  )
+  (wire (pts (xy 49.53 55.88) (xy 49.53 67.31))
+    (stroke (width 0) (type default) (color 0 0 0 0))
+  )
+  (wire (pts (xy 86.36 81.28) (xy 95.25 81.28))
+    (stroke (width 0) (type default) (color 0 0 0 0))
+  )
+  (wire (pts (xy 86.36 78.74) (xy 97.79 78.74))
+    (stroke (width 0) (type default) (color 0 0 0 0))
+  )
+  (wire (pts (xy 86.36 83.82) (xy 102.87 83.82))
+    (stroke (width 0) (type default) (color 0 0 0 0))
+  )
+  (wire (pts (xy 76.2 53.34) (xy 87.63 53.34))
+    (stroke (width 0) (type default) (color 0 0 0 0))
+  )
+  (wire (pts (xy 39.37 109.22) (xy 57.15 109.22))
+    (stroke (width 0) (type default) (color 0 0 0 0))
+  )
+  (wire (pts (xy 39.37 111.76) (xy 57.15 111.76))
+    (stroke (width 0) (type default) (color 0 0 0 0))
+  )
+  (wire (pts (xy 45.72 67.31) (xy 49.53 67.31))
+    (stroke (width 0) (type default) (color 0 0 0 0))
+  )
+  (wire (pts (xy 44.45 34.29) (xy 57.15 34.29))
+    (stroke (width 0) (type default) (color 0 0 0 0))
+  )
+  (wire (pts (xy 45.72 81.28) (xy 57.15 81.28))
+    (stroke (width 0) (type default) (color 0 0 0 0))
+  )
+  (wire (pts (xy 102.87 83.82) (xy 102.87 77.47))
+    (stroke (width 0) (type default) (color 0 0 0 0))
+  )
+  (wire (pts (xy 140.97 26.67) (xy 152.4 26.67))
+    (stroke (width 0) (type default) (color 0 0 0 0))
+  )
+  (wire (pts (xy 128.27 31.75) (xy 116.84 31.75))
+    (stroke (width 0) (type default) (color 0 0 0 0))
+  )
+  (wire (pts (xy 45.72 53.34) (xy 57.15 53.34))
+    (stroke (width 0) (type default) (color 0 0 0 0))
+  )
+  (wire (pts (xy 45.72 26.67) (xy 57.15 26.67))
+    (stroke (width 0) (type default) (color 0 0 0 0))
+  )
+  (wire (pts (xy 86.36 93.98) (xy 97.79 93.98))
+    (stroke (width 0) (type default) (color 0 0 0 0))
+  )
+  (wire (pts (xy 140.97 36.83) (xy 152.4 36.83))
+    (stroke (width 0) (type default) (color 0 0 0 0))
+  )
+  (wire (pts (xy 140.97 31.75) (xy 152.4 31.75))
+    (stroke (width 0) (type default) (color 0 0 0 0))
+  )
+  (wire (pts (xy 44.45 41.91) (xy 57.15 41.91))
+    (stroke (width 0) (type default) (color 0 0 0 0))
+  )
+  (wire (pts (xy 102.87 99.06) (xy 102.87 92.71))
+    (stroke (width 0) (type default) (color 0 0 0 0))
+  )
   (wire (pts (xy 140.97 34.29) (xy 152.4 34.29))
     (stroke (width 0) (type default) (color 0 0 0 0))
   )
-  (wire (pts (xy 76.2 35.56) (xy 87.63 35.56))
-    (stroke (width 0) (type default) (color 0 0 0 0))
-  )
-  (wire (pts (xy 49.53 55.88) (xy 57.15 55.88))
-    (stroke (width 0) (type default) (color 0 0 0 0))
-  )
-  (wire (pts (xy 45.72 78.74) (xy 57.15 78.74))
-    (stroke (width 0) (type default) (color 0 0 0 0))
-  )
-  (wire (pts (xy 49.53 55.88) (xy 49.53 67.31))
-    (stroke (width 0) (type default) (color 0 0 0 0))
-  )
-  (wire (pts (xy 86.36 81.28) (xy 95.25 81.28))
-    (stroke (width 0) (type default) (color 0 0 0 0))
-  )
-  (wire (pts (xy 86.36 78.74) (xy 97.79 78.74))
-    (stroke (width 0) (type default) (color 0 0 0 0))
-  )
-  (wire (pts (xy 86.36 83.82) (xy 102.87 83.82))
-    (stroke (width 0) (type default) (color 0 0 0 0))
-  )
-  (wire (pts (xy 76.2 53.34) (xy 87.63 53.34))
-    (stroke (width 0) (type default) (color 0 0 0 0))
-  )
-  (wire (pts (xy 39.37 109.22) (xy 57.15 109.22))
-    (stroke (width 0) (type default) (color 0 0 0 0))
-  )
-  (wire (pts (xy 39.37 111.76) (xy 57.15 111.76))
-    (stroke (width 0) (type default) (color 0 0 0 0))
-  )
-  (wire (pts (xy 45.72 67.31) (xy 49.53 67.31))
-    (stroke (width 0) (type default) (color 0 0 0 0))
-  )
-  (wire (pts (xy 44.45 34.29) (xy 57.15 34.29))
-    (stroke (width 0) (type default) (color 0 0 0 0))
-  )
-  (wire (pts (xy 45.72 81.28) (xy 57.15 81.28))
-    (stroke (width 0) (type default) (color 0 0 0 0))
-  )
-  (wire (pts (xy 102.87 83.82) (xy 102.87 77.47))
-    (stroke (width 0) (type default) (color 0 0 0 0))
-  )
-  (wire (pts (xy 140.97 26.67) (xy 152.4 26.67))
-    (stroke (width 0) (type default) (color 0 0 0 0))
-  )
-  (wire (pts (xy 128.27 31.75) (xy 116.84 31.75))
-    (stroke (width 0) (type default) (color 0 0 0 0))
-  )
-  (wire (pts (xy 45.72 53.34) (xy 57.15 53.34))
-    (stroke (width 0) (type default) (color 0 0 0 0))
-  )
-  (wire (pts (xy 45.72 26.67) (xy 57.15 26.67))
-    (stroke (width 0) (type default) (color 0 0 0 0))
-  )
-  (wire (pts (xy 86.36 93.98) (xy 97.79 93.98))
-    (stroke (width 0) (type default) (color 0 0 0 0))
-  )
-  (wire (pts (xy 140.97 31.75) (xy 152.4 31.75))
-    (stroke (width 0) (type default) (color 0 0 0 0))
-  )
-  (wire (pts (xy 140.97 36.83) (xy 152.4 36.83))
-    (stroke (width 0) (type default) (color 0 0 0 0))
-  )
-  (wire (pts (xy 102.87 99.06) (xy 102.87 92.71))
-    (stroke (width 0) (type default) (color 0 0 0 0))
-  )
   (wire (pts (xy 44.45 36.83) (xy 57.15 36.83))
     (stroke (width 0) (type default) (color 0 0 0 0))
@@
     (stroke (width 0) (type default) (color 0 0 0 0))
   )
+  (wire (pts (xy 44.45 39.37) (xy 57.15 39.37))
+    (stroke (width 0) (type default) (color 0 0 0 0))
+  )
   (wire (pts (xy 97.79 77.47) (xy 97.79 78.74))
     (stroke (width 0) (type default) (color 0 0 0 0))
@@
     (effects (font (size 1.27 1.27)) (justify left bottom))
   )
-  (label "sw0" (at 147.32 34.29 0)
+  (label "sw0" (at 116.84 41.91 0)
     (effects (font (size 1.27 1.27)) (justify left bottom))
   )
@@
     (effects (font (size 1.27 1.27)) (justify left bottom))
   )
+  (label "therm3" (at 152.4 34.29 180)
+    (effects (font (size 1.27 1.27)) (justify right bottom))
+  )
   (label "therm1" (at 49.53 36.83 0)
     (effects (font (size 1.27 1.27)) (justify left bottom))
@@
     (effects (font (size 1.27 1.27)) (justify left bottom))
   )
-  (label "fan1" (at 147.32 36.83 0)
-    (effects (font (size 1.27 1.27)) (justify left bottom))
+  (label "therm2" (at 57.15 39.37 180)
+    (effects (font (size 1.27 1.27)) (justify right bottom))
+  )
+  (label "fan1" (at 152.4 41.91 180)
+    (effects (font (size 1.27 1.27)) (justify right bottom))
   )
   (label "fan0" (at 118.11 36.83 0)
@@
     (effects (font (size 1.27 1.27)) (justify left bottom))
   )
+  (label "therm3" (at 57.15 41.91 180)
+    (effects (font (size 1.27 1.27)) (justify right bottom))
+  )
+  (label "therm2" (at 152.4 36.83 180)
+    (effects (font (size 1.27 1.27)) (justify right bottom))
+  )
   (label "VFAN1" (at 88.9 96.52 0)
     (effects (font (size 1.27 1.27)) (justify left bottom))
@@
   (symbol (lib_id "Connector:Conn_01x04_Female") (at 39.37 36.83 0) (mirror y) (unit 1)
     (in_bom yes) (on_board yes)
-    (property "Reference" "J?" (id 0) (at 39.37 31.75 0))
+    (property "Reference" "J3" (id 0) (at 39.37 31.75 0))
     (property "Value" "Conn_01x04_Female" (id 1) (at 39.37 44.45 0))
-    (property "Footprint" "Connector_JST:JST_PH_B2B-PH-K_1x02_P2.00mm_Vertical" (id 2) (at 39.37 36.83 0)
+    (property "Footprint" "Connector_JST:JST_PH_B4B-PH-K_1x04_P2.00mm_Vertical" (id 2) (at 39.37 36.83 0)
       (effects (font (size 1.27 1.27)) hide)
     )
@@
       (reference "J2") (unit 1) (value "Conn_01x02_Female") (footprint "Connector_Molex:Molex_Micro-Fit_3.0_43045-0200_2x01_P3.00mm_Horizontal")
     )
+    (path "/00000000-0000-0000-0000-000060d4eb4a"
+      (reference "J3") (unit 1) (value "Conn_01x04_Female") (footprint "Connector_JST:JST_PH_B4B-PH-K_1x04_P2.00mm_Vertical")
+    )
     (path "/00000000-0000-0000-0000-000060d4bb3b"
       (reference "J4") (unit 1) (value "Conn_01x02_Female") (footprint "Connector_JST:JST_PH_B2B-PH-K_1x02_P2.00mm_Vertical")
@@
       (reference "J11") (unit 1) (value "Conn_01x03_Female") (footprint "Jumper:SolderJumper-3_P1.3mm_Bridged12_RoundedPad1.0x1.5mm_NumberLabels")
     )
-    (path "/00000000-0000-0000-0000-000060d4eb4a"
-      (reference "J?") (unit 1) (value "Conn_01x04_Female") (footprint "Connector_JST:JST_PH_B2B-PH-K_1x02_P2.00mm_Vertical")
-    )
-  )
+  )

Commit message: Moved some things, added CT, checked clearance
Parts:
- added TH1: Thermistor_NTC, Resistor_THT:R_Axial_DIN0204_L3.6mm_D1.6mm_P7.62mm_Horizontal, symbol Device:Thermistor_NTC
Connections:
- net ctherm0: now reaches J9.1 (Pin_1)
- net ctherm0: now also TH1.1
- net ctherm1: now reaches J9.10 (Pin_10)
- net ctherm1: now also TH1.2
Other:
- moved on the sheet: J9
