File: v0_miniAB_batboard.kicad_pcb (KiCad board)
At the start: 2 copper layers, 51.5 x 37.4 mm, 16 parts, among them J1 Conn_01x04_Female, J10 Conn_01x03_Female, J11 Conn_01x03_Female, J2 Conn_01x02_Female, J3 Conn_01x04_Female, J4 Conn_01x02_Female, J5 Conn_01x02_Female, J6 Conn_01x02_Female, J7 Conn_01x03_Female, J8 Conn_01x03_Female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

Commit message: Minor adjustments and added Gerber files
Parts:
- J9: value Conn_02x07_Counter_Clockwise -> Conn_02x09_Counter_Clockwise
Changed lines of the file:
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@@
       (layerselection 0x00010fc_ffffffff)
       (disableapertmacros false)
-      (usegerberextensions false)
+      (usegerberextensions true)
       (usegerberattributes true)
       (usegerberadvancedattributes true)
@@
     (descr "Molex Micro-Fit 3.0 Connector System, 43045-0200 (alternative finishes: 43045-020x), 1 Pins per row (https://www.molex.com/pdm_docs/sd/430450201_sd.pdf), generated with kicad-footprint-generator")
     (tags "connector Molex Micro-Fit_3.0 horizontal")
-    (property "Sheetfile" "v0_miniAB_pancake_board.kicad_sch")
+    (property "Sheetfile" "v0_miniAB_batboard.kicad_sch")
     (property "Sheetname" "")
     (attr through_hole)
@@
     (descr "JST PH series connector, B4B-PH-K (http://www.jst-mfg.com/product/pdf/eng/ePH.pdf), generated with kicad-footprint-generator")
     (tags "connector JST PH side entry")
-    (property "Sheetfile" "v0_miniAB_pancake_board.kicad_sch")
+    (property "Sheetfile" "v0_miniAB_batboard.kicad_sch")
     (property "Sheetname" "")
     (attr through_hole)
@@
     (fp_line (start -2.36 -2.11) (end -2.36 -0.86) (layer "F.Fab") (width 0.1))
     (fp_line (start -1.95 -1.7) (end -1.95 2.8) (layer "F.Fab") (width 0.1))
-    (pad "1" thru_hole roundrect (at 0 0 90) (size 1.2 1.75) (drill 0.75) (layers *.Cu *.Mask) (roundrect_rratio 0.208333)
+    (pad "1" thru_hole roundrect (at 0 0 90) (size 1.2 1.75) (drill 0.75) (layers *.Cu *.Mask) (roundrect_rratio 0.2083333333)
       (net 6 "/therm0") (pinfunction "Pin_1") (pintype "passive"))
     (pad "2" thru_hole oval (at 2 0 90) (size 1.2 1.75) (drill 0.75) (layers *.Cu *.Mask)
@@
     (descr "JST PH series connector, B2B-PH-K (http://www.jst-mfg.com/product/pdf/eng/ePH.pdf), generated with kicad-footprint-generator")
     (tags "connector JST PH side entry")
-    (property "Sheetfile" "v0_miniAB_pancake_board.kicad_sch")
+    (property "Sheetfile" "v0_miniAB_batboard.kicad_sch")
     (property "Sheetname" "")
     (attr through_hole)
@@
     (descr "JST PH series connector, B3B-PH-K (http://www.jst-mfg.com/product/pdf/eng/ePH.pdf), generated with kicad-footprint-generator")
     (tags "connector JST PH side entry")
-    (property "Sheetfile" "v0_miniAB_pancake_board.kicad_sch")
+    (property "Sheetfile" "v0_miniAB_batboard.kicad_sch")
     (property "Sheetname" "")
     (attr through_hole)
@@
     (descr "JST PH series connector, B3B-PH-K (http://www.jst-mfg.com/product/pdf/eng/ePH.pdf), generated with kicad-footprint-generator")
     (tags "connector JST PH side entry")
-    (property "Sheetfile" "v0_miniAB_pancake_board.kicad_sch")
+    (property "Sheetfile" "v0_miniAB_batboard.kicad_sch")
     (property "Sheetname" "")
     (attr through_hole)
@@
     (descr "Molex Micro-Fit 3.0 Connector System, 43045-1800 (alternative finishes: 43045-180x), 9 Pins per row (https://www.molex.com/pdm_docs/sd/430450201_sd.pdf), generated with kicad-footprint-generator")
     (tags "connector Molex Micro-Fit_3.0 horizontal")
-    (property "Sheetfile" "v0_miniAB_pancake_board.kicad_sch")
+    (property "Sheetfile" "v0_miniAB_batboard.kicad_sch")
     (property "Sheetname" "")
     (attr through_hole)
@@
       (effects (font (size 1 1) (thickness 0.15)))
     )
-    (fp_text value "Conn_02x07_Counter_Clockwise" (at 12 5.7) (layer "F.Fab")
+    (fp_text value "Conn_02x09_Counter_Clockwise" (at 12 5.7) (layer "F.Fab")
       (effects (font (size 1 1) (thickness 0.15)))
     )
@@
       (effects (font (size 1 1) (thickness 0.15)))
     )
-    (fp_line (start 27.685 -8.03) (end 27.685 1.1) (layer "F.SilkS") (width 0.12))
     (fp_line (start -2.685 -9.03) (end 26.685 -9.03) (layer "F.SilkS") (width 0.12))
-    (fp_line (start -3.685 -8.03) (end -2.685 -9.03) (layer "F.SilkS") (width 0.12))
     (fp_line (start -3.685 1.1) (end -3.685 -8.03) (layer "F.SilkS") (width 0.12))
+    (fp_line (start 27.685 -8.03) (end 27.685 1.1) (layer "F.SilkS") (width 0.12))
+    (fp_line (start -3.685 -8.03) (end -2.685 -9.03) (layer "F.SilkS") (width 0.12))
     (fp_line (start 26.685 -9.03) (end 27.685 -8.03) (layer "F.SilkS") (width 0.12))
     (fp_line (start 27.685 1.1) (end -3.685 1.1) (layer "F.SilkS") (width 0.12))
-    (fp_line (start 28.08 -9.42) (end 28.08 1.49) (layer "F.CrtYd") (width 0.05))
-    (fp_line (start -1.25 4.25) (end -1.25 1.49) (layer "F.CrtYd") (width 0.05))
     (fp_line (start 25.25 4.25) (end -1.25 4.25) (layer "F.CrtYd") (width 0.05))
+    (fp_line (start -4.08 1.49) (end -4.08 -9.42) (layer "F.CrtYd") (width 0.05))
+    (fp_line (start -1.25 4.25) (end -1.25 1.49) (layer "F.CrtYd") (width 0.05))
+    (fp_line (start 25.25 1.49) (end 25.25 4.25) (layer "F.CrtYd") (width 0.05))
     (fp_line (start -4.08 -9.42) (end 28.08 -9.42) (layer "F.CrtYd") (width 0.05))
+    (fp_line (start 28.08 -9.42) (end 28.08 1.49) (layer "F.CrtYd") (width 0.05))
     (fp_line (start 28.08 1.49) (end 25.25 1.49) (layer "F.CrtYd") (width 0.05))
-    (fp_line (start -4.08 1.49) (end -4.08 -9.42) (layer "F.CrtYd") (width 0.05))
     (fp_line (start -1.25 1.49) (end -4.08 1.49) (layer "F.CrtYd") (width 0.05))
-    (fp_line (start 25.25 1.49) (end 25.25 4.25) (layer "F.CrtYd") (width 0.05))
-    (fp_line (start -3.575 -7.92) (end -2.575 -8.92) (layer "F.Fab") (width 0.1))
-    (fp_line (start -3.575 0.99) (end -3.575 -7.92) (layer "F.Fab") (width 0.1))
-    (fp_line (start 27.575 -7.92) (end 27.575 0.99) (layer "F.Fab") (width 0.1))
-    (fp_line (start 26.575 -8.92) (end 27.575 -7.92) (layer "F.Fab") (width 0.1))
-    (fp_line (start 27.575 0.99) (end -3.575 0.99) (layer "F.Fab") (width 0.1))
     (fp_line (start -0.75 0.99) (end 0 0) (layer "F.Fab") (width 0.1))
     (fp_line (start 0 0) (end 0.75 0.99) (layer "F.Fab") (width 0.1))
     (fp_line (start -2.575 -8.92) (end 26.575 -8.92) (layer "F.Fab") (width 0.1))
+    (fp_line (start 27.575 0.99) (end -3.575 0.99) (layer "F.Fab") (width 0.1))
+    (fp_line (start -3.575 -7.92) (end -2.575 -8.92) (layer "F.Fab") (width 0.1))
+    (fp_line (start 27.575 -7.92) (end 27.575 0.99) (layer "F.Fab") (width 0.1))
+    (fp_line (start -3.575 0.99) (end -3.575 -7.92) (layer "F.Fab") (width 0.1))
+    (fp_line (start 26.575 -8.92) (end 27.575 -7.92) (layer "F.Fab") (width 0.1))
     (pad "" np_thru_hole circle (at 21.86 -4.32) (size 3 3) (drill 3) (layers *.Cu *.Mask))
     (pad "" np_thru_hole circle (at 2.16 -4.32) (size 3 3) (drill 3) (layers *.Cu *.Mask))
-    (pad "1" thru_hole roundrect (at 0 0) (size 1.5 1.5) (drill 1.02) (layers *.Cu *.Mask) (roundrect_rratio 0.166667)
+    (pad "1" thru_hole roundrect (at 0 0) (size 1.5 1.5) (drill 1.02) (layers *.Cu *.Mask) (roundrect_rratio 0.1666673333)
       (net 17 "/ctherm0") (pinfunction "Pin_1") (pintype "passive"))
     (pad "2" thru_hole circle (at 3 0) (size 1.5 1.5) (drill 1.02) (layers *.Cu *.Mask)
@@
       (rotate (xyz 0 0 0))
     )
-    (model "${KIPRJMOD}/step/430451800.stp"
-      (offset (xyz 12 4 4))
-      (scale (xyz 1 1 1))
-      (rotate (xyz -90 0 180))
-    )
   )
   (footprint "Jumper:SolderJumper-3_P1.3mm_Bridged12_RoundedPad1.0x1.5mm_NumberLabels" (layer "F.Cu")
@@
     (descr "SMD Solder 3-pad Jumper, 1x1.5mm rounded Pads, 0.3mm gap, pads 1-2 bridged with 1 copper strip, labeled with numbers")
     (tags "solder jumper open")
-    (property "Sheetfile" "v0_miniAB_pancake_board.kicad_sch")
+    (property "Sheetfile" "v0_miniAB_batboard.kicad_sch")
     (property "Sheetname" "")
     (attr exclude_from_pos_files)
@@
     (descr "SMD Solder 3-pad Jumper, 1x1.5mm rounded Pads, 0.3mm gap, pads 1-2 bridged with 1 copper strip, labeled with numbers")
     (tags "solder jumper open")
-    (property "Sheetfile" "v0_miniAB_pancake_board.kicad_sch")
+    (property "Sheetfile" "v0_miniAB_batboard.kicad_sch")
     (property "Sheetname" "")
     (attr exclude_from_pos_files)
@@
     (descr "JST PH series connector, B4B-PH-K (http://www.jst-mfg.com/product/pdf/eng/ePH.pdf), generated with kicad-footprint-generator")
     (tags "connector JST PH side entry")
-    (property "Sheetfile" "v0_miniAB_pancake_board.kicad_sch")
+    (property "Sheetfile" "v0_miniAB_batboard.kicad_sch")
     (property "Sheetname" "")
     (attr through_hole)
@@
     (descr "JST PH series connector, B2B-PH-K (http://www.jst-mfg.com/product/pdf/eng/ePH.pdf), generated with kicad-footprint-generator")
     (tags "connector JST PH side entry")
-    (property "Sheetfile" "v0_miniAB_pancake_board.kicad_sch")
+    (property "Sheetfile" "v0_miniAB_batboard.kicad_sch")
     (property "Sheetname" "")
     (attr through_hole)
@@
     (descr "JST PH series connector, B2B-PH-K (http://www.jst-mfg.com/product/pdf/eng/ePH.pdf), generated with kicad-footprint-generator")
     (tags "connector JST PH side entry")
-    (property "Sheetfile" "v0_miniAB_pancake_board.kicad_sch")
+    (property "Sheetfile" "v0_miniAB_batboard.kicad_sch")
     (property "Sheetname" "")
     (attr through_hole)
@@
     (descr "Resistor, Axial_DIN0204 series, Axial, Horizontal, pin pitch=7.62mm, 0.167W, length*diameter=3.6*1.6mm^2, http://cdn-reichelt.de/documents/datenblatt/B400/1_4W%23YAG.pdf")
     (tags "Resistor Axial_DIN0204 series Axial Horizontal pin pitch 7.62mm 0.167W length 3.6mm diameter 1.6mm")
-    (property "Sheetfile" "v0_miniAB_pancake_board.kicad_sch")
+    (property "Sheetfile" "v0_miniAB_batboard.kicad_sch")
     (property "Sheetname" "")
     (attr through_hole)
@@
     (effects (font (size 1 1) (thickness 0.15)) (justify mirror))
   )
-  (gr_text "this side \ntowards stepper" (at 87.3 98.2 90) (layer "B.SilkS")
+  (gr_text "this side \ntowards stepper" (at 86.25 94.25 45) (layer "B.SilkS")
     (effects (font (size 1 1) (thickness 0.15)) (justify mirror))
   )
