File: v0_miniAB_batboard.kicad_sch (KiCad schematic)
At the start: 12 parts, among them J1 Conn_01x04_Female, J10 Conn_01x03_Female, J11 Conn_01x03_Female, J2 Conn_01x02_Female, J3 Conn_01x04_Female, J4 Conn_01x02_Female, J5 Conn_01x02_Female, J6 Conn_01x02_Female, J7 Conn_01x03_Female, J8 Conn_01x03_Female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

Commit message: Minor adjustments and added Gerber files
Parts:
- J9: value Conn_02x07_Counter_Clockwise -> Conn_02x09_Counter_Clockwise
Changed lines of the file:
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@@
     (in_bom yes) (on_board yes)
     (property "Reference" "J9" (id 0) (at 134.62 35.1282 0))
-    (property "Value" "Conn_02x07_Counter_Clockwise" (id 1) (at 134.62 33.02 0))
+    (property "Value" "Conn_02x09_Counter_Clockwise" (id 1) (at 134.62 33.02 0))
     (property "Footprint" "Connector_Molex:Molex_Micro-Fit_3.0_43045-1800_2x09_P3.00mm_Horizontal" (id 2) (at 133.35 48.26 0)
       (effects (font (size 1.27 1.27)) hide)
@@
     )
     (path "/00000000-0000-0000-0000-000060d59db3"
-      (reference "J9") (unit 1) (value "Conn_02x07_Counter_Clockwise") (footprint "Connector_Molex:Molex_Micro-Fit_3.0_43045-1800_2x09_P3.00mm_Horizontal")
+      (reference "J9") (unit 1) (value "Conn_02x09_Counter_Clockwise") (footprint "Connector_Molex:Molex_Micro-Fit_3.0_43045-1800_2x09_P3.00mm_Horizontal")
     )
     (path "/00000000-0000-0000-0000-0000612c0080"
